Commit message: Working PPO and isaacgym version. Starting moving mass task.

File: assets/robot_mvw.urdf (robot description, URDF)
Before this commit: robot cart, 6 links, 5 joints
Links:
- removed link pendulum
- added link payload, mass 18; collision box size=0.1 0.1 0.1; visual box size=0.1 0.1 0.1
Joints:
- removed joint pendulum
- added joint payload: type prismatic, parent cart_base, child payload, origin xyz=0 0 0.15694736842105264 rpy=0 0 0, axis 1 0 0, limit lower=-0.25 upper=0.25 effort=440 velocity=10

Commit message: Working test of terrain generation, scandot measure, and mass movement.

File: assets/robot_mvw.urdf (robot description, URDF)
Before this commit: robot cart, 6 links, 5 joints
Joints:
- joint cart_to_left_back_wheel: limit lower=-10000 upper=10000 effort=5 velocity=10 -> lower=-10000 upper=10000 effort=15 velocity=15
- joint cart_to_left_front_wheel: limit lower=-10000 upper=10000 effort=5 velocity=10 -> lower=-10000 upper=10000 effort=15 velocity=15
- joint cart_to_right_back_wheel: limit lower=-10000 upper=10000 effort=5 velocity=10 -> lower=-10000 upper=10000 effort=15 velocity=15
- joint cart_to_right_front_wheel: limit lower=-10000 upper=10000 effort=5 velocity=10 -> lower=-10000 upper=10000 effort=15 velocity=15

Commit message: Current working version of moving mass robot climbing a ledge.

File: assets/robot_mvw.urdf (robot description, URDF)
Before this commit: robot cart, 6 links, 5 joints
Joints:
- joint payload: limit lower=-0.25 upper=0.25 effort=440 velocity=10 -> lower=-0.25 upper=0.25 effort=100 velocity=10
